File: lime2_adapter/eagle/lime2_adapter.sch (EAGLE design)
At the start: 23 parts, among them T1 MOSFET-N-NX7002AK, T2 MOSFET-N-NX7002AK, X1 lcd0_d02, X2 D-SUB15-HDR15RA, X4 XF2-40-RARBT, X5 FPC40-525594052

Commit message: Realize ECOs from Luc 190508
- Change X1-02 (X1B) to be disconnected
- Change X1-04 (X1D) to be disconnected
- Change X1-06 (X1F) to be disconnected
- Change X1-07 (X1G) to GPIO1-38(PC24)
- Change X1-08 (X1H) to GPIO1-40(PC23)
- Change X1-12 (X1L) to be disconnected
- Change X1-20 (X1T) to be disconnected
Parts:
- X1: value lcd0_d02 -> LCD
Connections:
- net EINT15/NCE7/SPI2_MISO/PC22: no longer X1-20.MS
- net NC/IR0_RX/PB4: no longer X1-6.MS
- net NC/IR0_TX/SPDIF_MCLK/STANBYWFI/PB3: no longer X1-7.MS
- net NDQS/PC24: now also X1-7.MS; no longer X1-8.MS
- net SPI0_CS0/PC23: now also X1-8.MS; no longer X1-12.MS
- net TWI1_SCK/PB18: no longer X1-4.MS
- net TWI1_SDA/PB19: no longer X1-2.MS

Commit message: lime2_adapter
- Change VCC_CSI0 (Camera) from X4-2 to X4-3
- Connect X1-2 to GND.
- Provide access to TVOUT3, LINEIN[L|R] and FMIN[L|R]
- Provide access to MIC[1|2]
Parts:
- added JP1, JP2: JP1E, jumper:JP1E
- added SV2: (no value), con-lstb:MA06-1
Connections:
- removed net CSI0_IO0: X4-35.MS
- removed net GNDA: A20_OLINUXINO_LIME2_SHIELD_GPIO-1.4
- removed net N$24: X4-16.MS
- removed net N$25: X4-15.MS
- removed net N$26: X4-14.MS
- removed net N$27: X4-13.MS
- removed net N$30: X4-10.MS
- removed net N$31: X4-9.MS
- removed net N$32: X4-8.MS
- removed net N$33: X4-7.MS
- removed net N$34: X4-6.MS
- removed net N$36: X4-4.MS
- removed net N$37: X4-3.MS
- removed net N$39: X4-1.MSV
- removed net N$4: X4-36.MS
- removed net N$6: X4-34.MS
- removed net N$7: R10.1, X4-2.MS
- removed net N$8: X4-32.MS
- net FMINL: now also SV2.1
- net FMINR: now also SV2.2
- net GND: now also A20_OLINUXINO_LIME2_SHIELD_GPIO-1.4, JP1.1, JP2.1, SV2.4
- net HSDA/UART7_RX/PS2_SDA0/PI21: now also X4-35.MS
- net LINEINL: now also SV2.3
- net LINEINR: now also SV2.5
- net MICIN1: now also JP2.2
- net MICIN2: now also JP1.2
- net N$3: now also R10.1, X4-3.MS; no longer X4-37.MS
- net TVOUT3: now also SV2.6
Other:
- note added: "ADC_X1"
- note added: "ADC_X2"
- note added: "ADC_Y1"
- note added: "ADC_Y2"
- note added: "CSI-IO0"
- note added: "CSI1-RESET#"
- note added: "CSI1-STBY-EN"
- note added: "FMINL"
- note added: "FMINR"
- note added: "HPL"
- note added: "HPR"
- note added: "LINEINL"
- note added: "LINEINR"
- note added: "LRADC0"
- note added: "LRADC1"
- note added: "TWI1-SCK"
- note added: "TWI1-SDA"
- moved on the sheet: LSP3, R1, R10, R6, R7, X4-1, X4-10, X4-11, X4-12, X4-13, X4-14, X4-15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
